Commit message: [base] mods to build [description] mod for remote view

File: husky_description/urdf/decorations.urdf.xacro (robot description, xacro)
@@ -16,5 +16,5 @@
         <origin xyz="0 0 0" rpy="0 0 0" />
         <geometry>
-          <mesh filename="file://$(find husky_description)/meshes/top_chassis.dae" />
+          <mesh filename="package://husky_description/meshes/top_chassis.dae" />
         </geometry>
       </visual>
@@ -30,5 +30,5 @@
         <visual>
           <geometry>
-            <mesh filename="file://$(find husky_description)/meshes/user_rail.dae" />
+            <mesh filename="package://husky_description/meshes/user_rail.dae" />
           </geometry>
         </visual>
@@ -45,5 +45,5 @@
       <visual>
         <geometry>
-          <mesh filename="file://$(find husky_description)/meshes/bumper.dae" />
+          <mesh filename="package://husky_description/meshes/bumper.dae" />
         </geometry>
       </visual>
@@ -59,5 +59,5 @@
           <visual>
               <geometry>
-                  <mesh filename="file://$(find husky_description)/meshes/bumper_extension.dae" />
+                  <mesh filename="package://husky_description/meshes/bumper_extension.dae" />
               </geometry>
           </visual>
@@ -73,5 +73,5 @@
       <visual>
         <geometry>
-          <mesh filename="file://$(find husky_description)/meshes/bumper.dae" />
+          <mesh filename="package://husky_description/meshes/bumper.dae" />
         </geometry>
       </visual>
@@ -87,5 +87,5 @@
           <visual>
               <geometry>
-                  <mesh filename="file://$(find husky_description)/meshes/bumper_extension.dae" />
+                  <mesh filename="package://husky_description/meshes/bumper_extension.dae" />
               </geometry>
           </visual>
@@ -104,5 +104,5 @@
             <origin xyz="0 0 0" rpy="0 0 0" />
             <geometry>
-              <mesh filename="file://$(find husky_description)/meshes/large_top_plate.dae" />
+              <mesh filename="package://husky_description/meshes/large_top_plate.dae" />
             </geometry>
           </visual>
@@ -110,5 +110,5 @@
             <origin xyz="0 0 0" rpy="0 0 0"/>
             <geometry>
-              <mesh filename="file://$(find husky_description)/meshes/large_top_plate_collision.stl" />
+              <mesh filename="package://husky_description/meshes/large_top_plate_collision.stl" />
             </geometry>
           </collision>
@@ -138,5 +138,5 @@
             <origin xyz="0 0 0" rpy="0 0 0" />
             <geometry>
-              <mesh filename="file://$(find husky_description)/meshes/top_plate.dae" />
+              <mesh filename="package://husky_description/meshes/top_plate.dae" />
             </geometry>
           </visual>
@@ -144,5 +144,5 @@
             <origin xyz="0 0 0" rpy="0 0 0"/>
             <geometry>
-              <mesh filename="file://$(find husky_description)/meshes/top_plate.stl" />
+              <mesh filename="package://husky_description/meshes/top_plate.stl" />
             </geometry>
           </collision>

File: husky_description/urdf/husky_macro.urdf.xacro (robot description, xacro)
@@ -37,5 +37,5 @@
         <origin xyz="0 0 0" rpy="0 0 0" />
         <geometry>
-          <mesh filename="file://$(find husky_description)/meshes/base_link.dae" />
+          <mesh filename="package://husky_description/meshes/base_link.dae" />
         </geometry>
       </visual>

File: husky_description/urdf/wheel.urdf.xacro (robot description, xacro)
@@ -11,5 +11,5 @@
         <origin xyz="0 0 0" rpy="0 0 0" />
         <geometry>
-          <mesh filename="file://$(find husky_description)/meshes/wheel.dae" />
+          <mesh filename="package://husky_description/meshes/wheel.dae" />
         </geometry>
       </visual>
