Commit message: [husky_description] gazebo mesh fix

File: husky_description/urdf/accessories/sensor_arch.urdf.xacro (robot description, xacro)
@@ -7,5 +7,5 @@
              <visual>
                  <geometry>
-                     <mesh filename="package://husky_description/meshes/accessories/${size}_mm_sensor_arch.dae" />
+                     <mesh filename="${mesh_path}/accessories/${size}_mm_sensor_arch.dae" />
                  </geometry>
              </visual>
@@ -13,5 +13,5 @@
                  <origin xyz="0 0 0" rpy="0 0 0"/>
                  <geometry>
-                     <mesh filename="package://husky_description/meshes/accessories/${size}_mm_sensor_arch.dae" />
+                     <mesh filename="${mesh_path}/accessories/${size}_mm_sensor_arch.dae" />
                  </geometry>
              </collision>

File: husky_description/urdf/accessories/sick_lms1xx_mount.urdf.xacro (robot description, xacro)
@@ -33,5 +33,5 @@
         <geometry>
           <!-- Origin of this mesh is the base of the bracket. -->
-          <mesh filename="package://husky_description/meshes/accessories/lms1xx_mount.dae" />
+          <mesh filename="${mesh_path}/accessories/lms1xx_mount.dae" />
         </geometry>
       </visual>

File: husky_description/urdf/decorations.urdf.xacro (robot description, xacro)
@@ -16,5 +16,5 @@
         <origin xyz="0 0 0" rpy="0 0 0" />
         <geometry>
-          <mesh filename="package://husky_description/meshes/top_chassis.dae" />
+          <mesh filename="${mesh_path}/top_chassis.dae" />
         </geometry>
       </visual>
@@ -30,5 +30,5 @@
         <visual>
           <geometry>
-            <mesh filename="package://husky_description/meshes/user_rail.dae" />
+            <mesh filename="${mesh_path}/user_rail.dae" />
           </geometry>
         </visual>
@@ -45,5 +45,5 @@
       <visual>
         <geometry>
-          <mesh filename="package://husky_description/meshes/bumper.dae" />
+          <mesh filename="${mesh_path}/bumper.dae" />
         </geometry>
       </visual>
@@ -59,5 +59,5 @@
           <visual>
               <geometry>
-                  <mesh filename="package://husky_description/meshes/bumper_extension.dae" />
+                  <mesh filename="${mesh_path}/bumper_extension.dae" />
               </geometry>
           </visual>
@@ -73,5 +73,5 @@
       <visual>
         <geometry>
-          <mesh filename="package://husky_description/meshes/bumper.dae" />
+          <mesh filename="${mesh_path}/bumper.dae" />
         </geometry>
       </visual>
@@ -87,5 +87,5 @@
           <visual>
               <geometry>
-                  <mesh filename="package://husky_description/meshes/bumper_extension.dae" />
+                  <mesh filename="${mesh_path}/bumper_extension.dae" />
               </geometry>
           </visual>
@@ -104,5 +104,5 @@
             <origin xyz="0 0 0" rpy="0 0 0" />
             <geometry>
-              <mesh filename="package://husky_description/meshes/large_top_plate.dae" />
+              <mesh filename="${mesh_path}/large_top_plate.dae" />
             </geometry>
           </visual>
@@ -110,5 +110,5 @@
             <origin xyz="0 0 0" rpy="0 0 0"/>
             <geometry>
-              <mesh filename="package://husky_description/meshes/large_top_plate_collision.stl" />
+              <mesh filename="${mesh_path}/large_top_plate_collision.stl" />
             </geometry>
           </collision>
@@ -138,5 +138,5 @@
             <origin xyz="0 0 0" rpy="0 0 0" />
             <geometry>
-              <mesh filename="package://husky_description/meshes/top_plate.dae" />
+              <mesh filename="${mesh_path}/top_plate.dae" />
             </geometry>
           </visual>
@@ -144,5 +144,5 @@
             <origin xyz="0 0 0" rpy="0 0 0"/>
             <geometry>
-              <mesh filename="package://husky_description/meshes/top_plate.stl" />
+              <mesh filename="${mesh_path}/top_plate.stl" />
             </geometry>
           </collision>

File: husky_description/urdf/husky.urdf.xacro (robot description, xacro)
@@ -5,4 +5,5 @@
   <xacro:arg name="prefix" default="" />
   <xacro:arg name="gazebo_controllers" default="$(find husky_control)/config/control.yaml" />
+  <xacro:property name="mesh_path" value="package://husky_description/meshes" />
   <xacro:include filename="$(find husky_description)/urdf/husky_macro.urdf.xacro" />
   <!-- Load husky description -->

File: husky_description/urdf/husky_macro.urdf.xacro (robot description, xacro)
@@ -13,4 +13,7 @@
   <xacro:arg name="is_sim" default="false" />
   <xacro:arg name="urdf_extras" default="empty.urdf" />
+  <xacro:if value="$(arg is_sim)">
+    <xacro:property name="mesh_path" value="file://$(find husky_description)/meshes" />
+  </xacro:if>
   <!-- Included URDF/XACRO Files -->
   <xacro:include filename="$(find husky_description)/urdf/decorations.urdf.xacro" />
@@ -37,5 +40,5 @@
         <origin xyz="0 0 0" rpy="0 0 0" />
         <geometry>
-          <mesh filename="package://husky_description/meshes/base_link.dae" />
+          <mesh filename="${mesh_path}/base_link.dae" />
         </geometry>
       </visual>

File: husky_description/urdf/wheel.urdf.xacro (robot description, xacro)
@@ -11,5 +11,5 @@
         <origin xyz="0 0 0" rpy="0 0 0" />
         <geometry>
-          <mesh filename="package://husky_description/meshes/wheel.dae" />
+          <mesh filename="${mesh_path}/wheel.dae" />
         </geometry>
       </visual>
